File: mesp240_3Dpad/mesp240_3Dpad.kicad_sch (KiCad schematic)
At the start: 64 parts, among them J1 1.27P CNX, J2 1.27P CNX, J3 Piezo Connector, J4 VibroMotorConnector, Q1 MMBT3904, Q2 MMBT3904, SW1 Button DOWN, SW2 Button LEFT, SW3 Button Right, SW4 Button UP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

Commit message: Fixing stupid inverted Schmitt Trigger
Connections:
- net +3V3: now also U1.14 (VCC); no longer U1.7 (GND)
- net GND: now also U1.7 (GND); no longer U1.14 (VCC)
Other:
- moved on the sheet: U1G
Changed lines of the file:
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@@
     (pin "9")
   )
-  (symbol (lib_id "JLCPCBA:74HC14D") (at 247.65 138.43 180) (unit 7)
+  (symbol (lib_id "JLCPCBA:74HC14D") (at 247.65 138.43 0) (unit 7)
     (in_bom yes) (on_board yes) (fields_autoplaced)
     (property "Reference" "U1" (id 0) (at 241.8079 137.5215 0)
-      (effects (font (size 1.27 1.27)) (justify left))
+      (effects (font (size 1.27 1.27)) (justify right))
     )
     (property "Value" "74HC14D" (id 1) (at 241.8079 140.2966 0)
-      (effects (font (size 1.27 1.27)) (justify left))
+      (effects (font (size 1.27 1.27)) (justify right))
     )
     (property "Footprint" "Package_SO:SOIC-14_3.9x8.7mm_P1.27mm" (id 2) (at 247.65 138.43 0)
@@
     (pin "14")
     (pin "7")
+  )
+  (symbol (lib_id "Connector:Conn_01x24_Male") (at 53.34 161.29 0) (unit 1)
+    (in_bom yes) (on_board yes)
+    (property "Reference" "J2" (id 0) (at 57.15 128.27 0)
+      (effects (font (size 1.27 1.27)) (justify right))
+    )
+    (property "Value" "1.27P CNX" (id 1) (at 58.42 130.81 0)
+      (effects (font (size 1.27 1.27)) (justify right))
+    )
+    (property "Footprint" "Connector_PinSocket_1.27mm:PinSocket_1x24_P1.27mm_Vertical" (id 2) (at 53.34 161.29 0)
+      (effects (font (size 1.27 1.27)) hide)
+    )
+    (property "Datasheet" "~" (id 3) (at 53.34 161.29 0)
+      (effects (font (size 1.27 1.27)) hide)
+    )
+    (property "LCSC" "" (id 4) (at 53.34 161.29 0)
+      (effects (font (size 1.27 1.27)) hide)
+    )
+    (pin "1")
+    (pin "10")
+    (pin "11")
+    (pin "12")
+    (pin "13")
+    (pin "14")
+    (pin "15")
+    (pin "16")
+    (pin "17")
+    (pin "18")
+    (pin "19")
+    (pin "2")
+    (pin "20")
+    (pin "21")
+    (pin "22")
+    (pin "23")
+    (pin "24")
+    (pin "3")
+    (pin "4")
+    (pin "5")
+    (pin "6")
+    (pin "7")
+    (pin "8")
+    (pin "9")
   )
   (symbol (lib_id "JLCPCBA:3D161") (at 177.8 91.44 0) (unit 1)
@@
     (pin "Y3")
   )
-  (symbol (lib_id "Connector:Conn_01x24_Male") (at 53.34 161.29 0) (unit 1)
-    (in_bom yes) (on_board yes)
-    (property "Reference" "J2" (id 0) (at 57.15 128.27 0)
-      (effects (font (size 1.27 1.27)) (justify right))
-    )
-    (property "Value" "1.27P CNX" (id 1) (at 58.42 130.81 0)
-      (effects (font (size 1.27 1.27)) (justify right))
-    )
-    (property "Footprint" "Connector_PinSocket_1.27mm:PinSocket_1x24_P1.27mm_Vertical" (id 2) (at 53.34 161.29 0)
-      (effects (font (size 1.27 1.27)) hide)
-    )
-    (property "Datasheet" "~" (id 3) (at 53.34 161.29 0)
-      (effects (font (size 1.27 1.27)) hide)
-    )
-    (property "LCSC" "" (id 4) (at 53.34 161.29 0)
-      (effects (font (size 1.27 1.27)) hide)
-    )
-    (pin "1")
-    (pin "10")
-    (pin "11")
-    (pin "12")
-    (pin "13")
-    (pin "14")
-    (pin "15")
-    (pin "16")
-    (pin "17")
-    (pin "18")
-    (pin "19")
-    (pin "2")
-    (pin "20")
-    (pin "21")
-    (pin "22")
-    (pin "23")
-    (pin "24")
-    (pin "3")
-    (pin "4")
-    (pin "5")
-    (pin "6")
-    (pin "7")
-    (pin "8")
-    (pin "9")
-  )
   (symbol (lib_id "Sensor_Motion:MPU-6050") (at 200.66 46.99 0) (unit 1)
